Commit message: backup

File: dh_ag95_description/urdf/dh_ag95.urdf.xacro (robot description, xacro)
@@ -23,4 +23,3 @@
         mock_sensor_commands="$(arg mock_sensor_commands)"
     />
-    <link name="world" />
 </robot>

Commit message: add gripper activation timeout + fix launch file

File: dh_ag95_description/urdf/dh_ag95.urdf.xacro (robot description, xacro)
@@ -9,4 +9,5 @@
     <xacro:include filename="$(find dh_ag95_description)/urdf/dh_ag95_macro.xacro" />
     <xacro:include filename="$(find dh_gripper_driver)/urdf/dh_ag95.ros2_control.xacro" />
+    <link name="world" />
     <!-- gripper -->
     <xacro:dh_ag95_gripper
